File: hardware/TRX_Board.kicad_sch (KiCad schematic)
At the start: 61 parts, among them J1 Conn_02x08_Odd_Even, J2 SMA, J3 Conn_01x03, J4 Conn_01x03, J5 Conn_01x03, Q1 BSN20, Q2 BSN20, Q3 BSN20, U1 AP1117-33, U2 LM386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

Commit message: Added missing parts sources
Parts:
- J1: Remarks (none) -> Mouser: 571-5-146268-8
- J2: Remarks (none) -> Mouser: 538-73391-0070
- J3, J4: Remarks (none) -> Mouser: 649-54201-G0803ALF
Changed lines of the file:
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@@
       (effects (font (size 1.27 1.27)) hide)
     )
-    (property "Datasheet" " ~" (id 3) (at 142.875 47.625 0)
+    (property "Datasheet" "https://www.mouser.ch/datasheet/2/276/3/0733910070_RF_COAX_CONNECTORS-2833758.pdf" (id 3) (at 142.875 47.625 0)
+      (effects (font (size 1.27 1.27)) hide)
+    )
+    (property "Remarks" "Mouser: 538-73391-0070" (id 4) (at 142.875 47.625 0)
       (effects (font (size 1.27 1.27)) hide)
     )
@@
       (effects (font (size 1.27 1.27)) hide)
     )
-    (property "Datasheet" "~" (id 3) (at 197.485 26.035 0)
+    (property "Datasheet" "https://cdn.amphenol-icc.com/media/wysiwyg/files/drawing/54201.pdf" (id 3) (at 197.485 26.035 0)
+      (effects (font (size 1.27 1.27)) hide)
+    )
+    (property "Remarks" "Mouser: 649-54201-G0803ALF" (id 4) (at 197.485 26.035 0)
       (effects (font (size 1.27 1.27)) hide)
     )
@@
       (effects (font (size 1.27 1.27)) hide)
     )
-    (property "Datasheet" "~" (id 3) (at 131.445 121.285 0)
+    (property "Datasheet" "https://www.mouser.ch/datasheet/2/418/6/ENG_CD_146268_H_146268_1_c_dwg-2007756.pdf" (id 3) (at 131.445 121.285 0)
+      (effects (font (size 1.27 1.27)) hide)
+    )
+    (property "Remarks" "Mouser: 571-5-146268-8" (id 4) (at 131.445 121.285 0)
       (effects (font (size 1.27 1.27)) hide)
     )
@@
       (effects (font (size 1.27 1.27)) hide)
     )
-    (property "Datasheet" "~" (id 3) (at 165.1 26.035 0)
-      (effects (font (size 1.27 1.27)) hide)
-    )
+    (property "Datasheet" "https://cdn.amphenol-icc.com/media/wysiwyg/files/drawing/54201.pdf" (id 3) (at 165.1 26.035 0)
+      (effects (font (size 1.27 1.27)) hide)
+    )
+    (property "Remarks" "Mouser: 649-54201-G0803ALF" (id 4) (at 165.1 26.035 0)
+      (effects (font (size 1.27 1.27)) hide)
+    )
